File: AE-001_Analog_Sensing_Supply/test.sch (KiCad schematic (older format))
At the start: 0 parts

Commit message: lucky test edit test.sch
Parts:
- added R?: R_PHOTO, symbol Device:R_PHOTO
Changed lines of the file:
@@
 Comment4 ""
 $EndDescr
+$Comp
+L Device:R_PHOTO R?
+U 1 1 5F1A4CA4
+P 5250 3900
+F 0 "R?" H 5320 3946 50  0000 L CNN
+F 1 "R_PHOTO" H 5320 3855 50  0000 L CNN
+F 2 "" V 5300 3650 50  0001 L CNN
+F 3 "~" H 5250 3850 50  0001 C CNN
+	1    5250 3900
+	1    0    0    -1
+$EndComp
 $EndSCHEMATC
