File: AE-001_Analog_Sensing_Supply/PS3.sch (KiCad schematic (older format))
At the start: 0 parts

Commit message: le buck
Parts:
- added CBOOST: C_0.1uF, footprints:C_0805_OEM, symbol formula:C_0.1uF
- added Cin (x2), Cout (x2): C_10uF, footprints:C_0805_OEM, symbol formula:C_10uF
- added Cvcc: C_1uF, footprints:C_0805_OEM, symbol formula:C_1uF
- added D: LED, symbol Device:LED
- added L1: L_15uH, footprints:L_100uH_OEM, symbol formula:L_15uH
- added R: R_2, symbol formula:R_2
- added Ren: R_1M, footprints:R_0805_OEM, symbol formula:R_1M
- added U: MCP16312, symbol formula:MCP16312
Connections:
- net labels added: GND
- wire segments 0 -> 15
