File: AE-001_Analog_Sensing_Supply/PS3.sch (KiCad schematic (older format))
At the start: 11 parts

Commit message: le fresh buck
Parts:
- removed CBOOST: C_0.1uF, footprints:C_0805_OEM, symbol formula:C_0.1uF
- removed D: LED, symbol Device:LED
- removed L1: L_15uH, footprints:L_100uH_OEM, symbol formula:L_15uH
- removed R: R_2, symbol formula:R_2
- removed Ren: R_1M, footprints:R_0805_OEM, symbol formula:R_1M
- added C_BOOST: C_100nF, footprints:C_0603_1608Metric, symbol formula:C_100nF
- added L1: L_22uH, symbol formula:L_22uH
- added R1: R_10K, footprints:R_0805_OEM, symbol formula:R_10K
- added R2: R_52.3k, symbol formula:R_52.3k
- renumbered Cin to C_IN1, Cin to C_IN2, Cout to C_OUT1, Cout to C_OUT2, Cvcc to C_VCC
Connections:
- net labels added: GNDA, GNDPWR
- wire segments 15 -> 32

Commit message: updated buck
Connections:
- net labels added: V_IN, V_OUT
- net labels removed: GND
- wire segments 32 -> 22
Changed lines of the file:
@@
 	3150 1400 3150 1200
-$Comp
-L power:GND #PWR?
-U 1 1 5F36A312
-P 2250 2500
-F 0 "#PWR?" H 2250 2250 50  0001 C CNN
-F 1 "GND" H 2255 2327 50  0000 C CNN
-F 2 "" H 2250 2500 50  0001 C CNN
-F 3 "" H 2250 2500 50  0001 C CNN
-	1    2250 2500
-	1    0    0    -1
-$EndComp
 $Comp
 L formula:C_1uF C_VCC
@@
 Wire Wire Line
 	2100 1950 2100 1700
-Connection ~ 2100 1700
-Wire Wire Line
-	2100 1700 1650 1700
 Wire Wire Line
 	3750 1800 3850 1800
@@
 Wire Wire Line
 	2500 1700 2100 1700
-$Comp
-L power:GND #PWR?
-U 1 1 5F35E286
-P 5000 2500
-F 0 "#PWR?" H 5000 2250 50  0001 C CNN
-F 1 "GND" H 5005 2327 50  0000 C CNN
-F 2 "" H 5000 2500 50  0001 C CNN
-F 3 "" H 5000 2500 50  0001 C CNN
-	1    5000 2500
-	1    0    0    -1
-$EndComp
 $Comp
 L formula:C_10uF C_OUT2
@@
 $EndComp
 $Comp
-L power:GND #PWR?
-U 1 1 5F37B41E
-P 1650 2500
-F 0 "#PWR?" H 1650 2250 50  0001 C CNN
-F 1 "GND" H 1655 2327 50  0000 C CNN
-F 2 "" H 1650 2500 50  0001 C CNN
-F 3 "" H 1650 2500 50  0001 C CNN
-	1    1650 2500
-	1    0    0    -1
-$EndComp
-$Comp
 L formula:C_10uF C_IN1
 U 1 1 5F36CAFB
@@
 	-1   0    0    1
 $EndComp
-Wire Wire Line
-	1500 2350 1500 2450
-Wire Wire Line
-	1500 2450 1650 2450
-Wire Wire Line
-	1800 2450 1800 2350
-Wire Wire Line
-	1650 2500 1650 2450
-Connection ~ 1650 2450
-Wire Wire Line
-	1650 2450 1800 2450
-Wire Wire Line
-	1650 1950 1500 1950
-Wire Wire Line
-	1500 1950 1500 2050
-Wire Wire Line
-	1650 1700 1650 1950
-Wire Wire Line
-	1650 1950 1800 1950
-Wire Wire Line
-	1800 1950 1800 2050
-Connection ~ 1650 1950
-Wire Wire Line
-	4850 2050 4850 1950
-Wire Wire Line
-	5150 1950 5150 2050
-Wire Wire Line
-	4850 1950 5000 1950
-Wire Wire Line
-	5000 1950 5000 1800
-Wire Wire Line
-	4250 1800 5000 1800
-Connection ~ 5000 1950
-Wire Wire Line
-	5000 1950 5150 1950
-Wire Wire Line
-	4850 2350 4850 2450
-Wire Wire Line
-	4850 2450 5000 2450
-Wire Wire Line
-	5150 2450 5150 2350
-Wire Wire Line
-	5000 2500 5000 2450
-Connection ~ 5000 2450
-Wire Wire Line
-	5000 2450 5150 2450
 Connection ~ 3850 1800
 $Comp
@@
 	1    0    0    -1
 $EndComp
-$Comp
-L power:GND #PWR?
-U 1 1 5F3A271E
-P 4250 2500
-F 0 "#PWR?" H 4250 2250 50  0001 C CNN
-F 1 "GND" H 4255 2327 50  0000 C CNN
-F 2 "" H 4250 2500 50  0001 C CNN
-F 3 "" H 4250 2500 50  0001 C CNN
-	1    4250 2500
-	1    0    0    -1
-$EndComp
 Wire Wire Line
 	3750 2100 4250 2100
@@
 	4250 2100 4250 2200
 Connection ~ 4250 2200
-Connection ~ 4250 1800
 $Comp
 L formula:R_52.3k R2
@@
 	1    0    0    -1
 $EndComp
+Wire Wire Line
+	4250 1800 4850 1800
+Wire Wire Line
+	4850 1800 4850 2050
+Connection ~ 4250 1800
+Wire Wire Line
+	4850 1800 5150 1800
+Wire Wire Line
+	5150 1800 5150 2050
+Connection ~ 4850 1800
+Wire Wire Line
+	2100 1700 1800 1700
+Wire Wire Line
+	1800 1700 1800 2050
+Connection ~ 2100 1700
+Wire Wire Line
+	1800 1700 1500 1700
+Wire Wire Line
+	1500 1700 1500 2050
+Connection ~ 1800 1700
+Wire Wire Line
+	1500 2350 1500 2500
+Wire Wire Line
+	1800 2350 1800 2500
+Wire Wire Line
+	4850 2350 4850 2500
+Wire Wire Line
+	5150 2350 5150 2500
+Text Label 5150 1800 0    50   ~ 0
+V_OUT
+Text Label 1500 1700 2    50   ~ 0
+V_IN
+$Comp
+L power:GNDA #PWR?
+U 1 1 5F4BA01E
+P 1500 2500
+F 0 "#PWR?" H 1500 2250 50  0001 C CNN
+F 1 "GNDA" H 1505 2327 50  0000 C CNN
+F 2 "" H 1500 2500 50  0001 C CNN
+F 3 "" H 1500 2500 50  0001 C CNN
+	1    1500 2500
+	1    0    0    -1
+$EndComp
+$Comp
+L power:GNDA #PWR?
+U 1 1 5F4C444F
+P 1800 2500
+F 0 "#PWR?" H 1800 2250 50  0001 C CNN
+F 1 "GNDA" H 1805 2327 50  0000 C CNN
+F 2 "" H 1800 2500 50  0001 C CNN
+F 3 "" H 1800 2500 50  0001 C CNN
+	1    1800 2500
+	1    0    0    -1
+$EndComp
+$Comp
+L power:GNDA #PWR?
+U 1 1 5F4C4935
+P 2250 2500
+F 0 "#PWR?" H 2250 2250 50  0001 C CNN
+F 1 "GNDA" H 2255 2327 50  0000 C CNN
+F 2 "" H 2250 2500 50  0001 C CNN
+F 3 "" H 2250 2500 50  0001 C CNN
+	1    2250 2500
+	1    0    0    -1
+$EndComp
+$Comp
+L power:GNDA #PWR?
+U 1 1 5F4C4EC2
+P 4250 2500
+F 0 "#PWR?" H 4250 2250 50  0001 C CNN
+F 1 "GNDA" H 4255 2327 50  0000 C CNN
+F 2 "" H 4250 2500 50  0001 C CNN
+F 3 "" H 4250 2500 50  0001 C CNN
+	1    4250 2500
+	1    0    0    -1
+$EndComp
+$Comp
+L power:GNDA #PWR?
+U 1 1 5F4C6950
+P 4850 2500
+F 0 "#PWR?" H 4850 2250 50  0001 C CNN
+F 1 "GNDA" H 4855 2327 50  0000 C CNN
+F 2 "" H 4850 2500 50  0001 C CNN
+F 3 "" H 4850 2500 50  0001 C CNN
+	1    4850 2500
+	1    0    0    -1
+$EndComp
+$Comp
+L power:GNDA #PWR?
+U 1 1 5F4C6F6B
+P 5150 2500
+F 0 "#PWR?" H 5150 2250 50  0001 C CNN
+F 1 "GNDA" H 5155 2327 50  0000 C CNN
+F 2 "" H 5150 2500 50  0001 C CNN
+F 3 "" H 5150 2500 50  0001 C CNN
+	1    5150 2500
+	1    0    0    -1
+$EndComp

Commit message: updated buck ground labels
Parts:
- C_BOOST: symbol formula:C_100nF -> PS3-rescue:C_100nF-formula
- L1: symbol formula:L_22uH -> PS3-rescue:L_22uH-formula
- R1: symbol formula:R_10K -> PS3-rescue:R_10K-formula
- R2: symbol formula:R_52.3k -> PS3-rescue:R_52.3k-formula
- U: symbol formula:MCP16312 -> PS3-rescue:MCP16312-formula
Changed lines of the file:
@@
 	3150 1200 3850 1200
 $Comp
-L formula:MCP16312 U
+L PS3-rescue:MCP16312-formula U
 U 1 1 5F3504EF
 P 3700 3150
@@
 $EndComp
 $Comp
-L formula:C_100nF C_BOOST
+L PS3-rescue:C_100nF-formula C_BOOST
 U 1 1 5F430872
 P 3850 1350
@@
 Connection ~ 3850 1800
 $Comp
-L formula:L_22uH L1
+L PS3-rescue:L_22uH-formula L1
 U 1 1 5F475F58
 P 4050 1750
@@
 $EndComp
 $Comp
-L formula:R_10K R1
+L PS3-rescue:R_10K-formula R1
 U 1 1 5F401EB3
 P 4250 2350
@@
 Connection ~ 4250 2200
 $Comp
-L formula:R_52.3k R2
+L PS3-rescue:R_52.3k-formula R2
 U 1 1 5F41CC0E
 P 4250 2000
@@
 $Comp
 L power:GNDA #PWR?
-U 1 1 5F4BA01E
-P 1500 2500
-F 0 "#PWR?" H 1500 2250 50  0001 C CNN
-F 1 "GNDA" H 1505 2327 50  0000 C CNN
-F 2 "" H 1500 2500 50  0001 C CNN
-F 3 "" H 1500 2500 50  0001 C CNN
-	1    1500 2500
-	1    0    0    -1
-$EndComp
-$Comp
-L power:GNDA #PWR?
-U 1 1 5F4C444F
-P 1800 2500
-F 0 "#PWR?" H 1800 2250 50  0001 C CNN
-F 1 "GNDA" H 1805 2327 50  0000 C CNN
-F 2 "" H 1800 2500 50  0001 C CNN
-F 3 "" H 1800 2500 50  0001 C CNN
-	1    1800 2500
-	1    0    0    -1
-$EndComp
-$Comp
-L power:GNDA #PWR?
 U 1 1 5F4C4935
 P 2250 2500
@@
 $EndComp
 $Comp
-L power:GNDA #PWR?
-U 1 1 5F4C6950
+L power:GNDPWR #PWR?
+U 1 1 5F4956B2
+P 1500 2500
+F 0 "#PWR?" H 1500 2300 50  0001 C CNN
+F 1 "GNDPWR" H 1422 2346 50  0000 C CNN
+F 2 "" H 1500 2450 50  0001 C CNN
+F 3 "" H 1500 2450 50  0001 C CNN
+	1    1500 2500
+	1    0    0    -1
+$EndComp
+$Comp
+L power:GNDPWR #PWR?
+U 1 1 5F495BD7
 P 4850 2500
-F 0 "#PWR?" H 4850 2250 50  0001 C CNN
-F 1 "GNDA" H 4855 2327 50  0000 C CNN
-F 2 "" H 4850 2500 50  0001 C CNN
-F 3 "" H 4850 2500 50  0001 C CNN
+F 0 "#PWR?" H 4850 2300 50  0001 C CNN
+F 1 "GNDPWR" H 4772 2346 50  0000 C CNN
+F 2 "" H 4850 2450 50  0001 C CNN
+F 3 "" H 4850 2450 50  0001 C CNN
 	1    4850 2500
 	1    0    0    -1
 $EndComp
 $Comp
-L power:GNDA #PWR?
-U 1 1 5F4C6F6B
+L power:GNDPWR #PWR?
+U 1 1 5F49D2AB
+P 1800 2500
+F 0 "#PWR?" H 1800 2300 50  0001 C CNN
+F 1 "GNDPWR" H 1804 2346 50  0000 C CNN
+F 2 "" H 1800 2450 50  0001 C CNN
+F 3 "" H 1800 2450 50  0001 C CNN
+	1    1800 2500
+	1    0    0    -1
+$EndComp
+$Comp
+L power:GNDPWR #PWR?
+U 1 1 5F4A200B
 P 5150 2500
-F 0 "#PWR?" H 5150 2250 50  0001 C CNN
-F 1 "GNDA" H 5155 2327 50  0000 C CNN
-F 2 "" H 5150 2500 50  0001 C CNN
-F 3 "" H 5150 2500 50  0001 C CNN
+F 0 "#PWR?" H 5150 2300 50  0001 C CNN
+F 1 "GNDPWR" H 5154 2346 50  0000 C CNN
+F 2 "" H 5150 2450 50  0001 C CNN
+F 3 "" H 5150 2450 50  0001 C CNN
 	1    5150 2500
 	1    0    0    -1

Commit message: buck layout v1
Parts:
- removed L1: L_22uH, symbol PS3-rescue:L_22uH-formula
- removed R2: R_52.3k, symbol PS3-rescue:R_52.3k-formula
- added L1: L_22uH, footprints:SRN8040, symbol formula:L_22uH
- added R2: R_52.3K, footprints:R_0805_OEM, symbol formula:R_52.3K
- C_BOOST1: renamed from C_BOOST; symbol PS3-rescue:C_100nF-formula -> formula:C_100nF
- R1: symbol PS3-rescue:R_10K-formula -> formula:R_10K
- U1: renamed from U; footprint (none) -> footprints:MCP16312; symbol PS3-rescue:MCP16312-formula -> formula:MCP16312; Purchasing Link (none) -> https://www.digikey.com/product-detail/en/microchip-technol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
- renumbered C_VCC to C_VCC1
Connections:
- wire segments 22 -> 35

Commit message: updated schematic with correct parts and links
Parts:
- L1: Purchasing Link (none) -> https://www.digikey.com/en/products/detail/kemet/L0805B220M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
- R2: symbol formula:R_52.3K -> formula:R_52.3k; Purchasing Link (none) -> https://www.digikey.com/en/products/detail/panasonic-electr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
- U1: footprint footprints:MCP16312 -> (none)
Connections:
- wire segments 35 -> 31
