File: AE-001_Analog_Sensing_Supply/PS2.sch (KiCad schematic (older format))
At the start: 9 parts

Commit message: Updated PS2
Parts:
- removed D?: BAT400D-7-F, symbol Formula:BAT400D-7-F
- removed R?: R_63.4, footprints:R_0805_OEM, symbol Formula:R_63.4
- added D1: CDBA140-G, symbol Formula:CDBA140-G
- added R1: R_6.2M, footprints:R_0805_OEM, symbol Formula:R_6.2M
- gave numbers to parts that had none: 7
Connections:
- wire segments 25 -> 28

Commit message: ps2 changes
Parts:
- removed R1: R_6.2M, footprints:R_0805_OEM, symbol Formula:R_6.2M
- added R1: R_7.5M, footprints:R_0805_OEM, symbol AE-001_Analog_Sensing_Supply-rescue:R_7.5M-Formula
- C1: symbol Formula:C_4.7uF_25V -> AE-001_Analog_Sensing_Supply-rescue:C_4.7uF_25V-Formula
- C2: symbol Formula:C_10nF -> AE-001_Analog_Sensing_Supply-rescue:C_10nF-Formula
- C3: symbol Formula:C_10uF -> AE-001_Analog_Sensing_Supply-rescue:C_10uF-Formula
- D1: symbol Formula:CDBA140-G -> AE-001_Analog_Sensing_Supply-rescue:CDBA140-G-Formula
- L1: symbol Formula:L_2.2uH -> AE-001_Analog_Sensing_Supply-rescue:L_2.2uH-Formula
- R2: symbol Formula:R_49.9K -> AE-001_Analog_Sensing_Supply-rescue:R_49.9K-Formula
- R3: symbol Formula:R_9.53K -> AE-001_Analog_Sensing_Supply-rescue:R_9.53K-Formula
- U1: symbol Formula:AOZ1280 -> AE-001_Analog_Sensing_Supply-rescue:AOZ1280-Formula
Changed lines of the file:
@@
 $EndDescr
 $Comp
-L Formula:C_4.7uF_25V C1
+L AE-001_Analog_Sensing_Supply-rescue:C_4.7uF_25V-Formula C1
 U 1 1 5F3028AB
 P 2700 3350
@@
 $EndComp
 $Comp
-L Formula:C_10uF C3
+L AE-001_Analog_Sensing_Supply-rescue:C_10uF-Formula C3
 U 1 1 5F303155
 P 6100 3800
@@
 $EndComp
 $Comp
-L Formula:C_10nF C2
+L AE-001_Analog_Sensing_Supply-rescue:C_10nF-Formula C2
 U 1 1 5F2D5B34
 P 4300 3100
@@
 $EndComp
 $Comp
-L Formula:L_2.2uH L1
+L AE-001_Analog_Sensing_Supply-rescue:L_2.2uH-Formula L1
 U 1 1 5F2D542D
 P 5250 3550
@@
 VOUT
 $Comp
-L Formula:R_9.53K R3
+L AE-001_Analog_Sensing_Supply-rescue:R_9.53K-Formula R3
 U 1 1 5F2F6E97
 P 5550 4100
@@
 	6100 3900 6100 4250
 $Comp
-L Formula:R_49.9K R2
+L AE-001_Analog_Sensing_Supply-rescue:R_49.9K-Formula R2
 U 1 1 5F2ED8B6
 P 5550 3750
@@
 	2700 3200 3200 3200
 $Comp
-L Formula:R_6.2M R1
-U 1 1 5F404635
-P 3200 3400
-F 0 "R1" H 3270 3446 50  0000 L CNN
-F 1 "R_6.2M" H 3270 3355 50  0000 L CNN
-F 2 "footprints:R_0805_OEM" H 2100 3700 50  0001 L CNN
-F 3 "https://www.vishay.com/docs/20035/dcrcwe3.pdf" H 2100 3800 50  0001 L CNN
-F 4 "https://www.digikey.com/product-detail/en/vishay-dale/CRCW08056M20FKEA/541-6-20MCTR-ND/1176107" H 2100 3900 60  0001 L CNN "PurchasingLink"
-	1    3200 3400
-	1    0    0    -1
-$EndComp
-$Comp
-L Formula:CDBA140-G D1
+L AE-001_Analog_Sensing_Supply-rescue:CDBA140-G-Formula D1
 U 1 1 5F405057
 P 4700 3800
@@
 $EndComp
 $Comp
-L Formula:AOZ1280 U1
+L AE-001_Analog_Sensing_Supply-rescue:AOZ1280-Formula U1
 U 1 1 5F2ED2E8
 P 3900 3500
+AR Path="/5F2ED2E8" Ref="U1"  Part="1"
+AR Path="/5F2CB8F1/5F2ED2E8" Ref="U1"  Part="1"
 F 0 "U1" H 3900 3750 50  0000 C CNN
 F 1 "AOZ1280" H 3600 2950 50  0000 C CNN
@@
 Wire Wire Line
 	4450 3100 4700 3100
+$Comp
+L AE-001_Analog_Sensing_Supply-rescue:R_7.5M-Formula R1
+U 1 1 5F48DE6E
+P 3200 3400
+F 0 "R1" H 3270 3446 50  0000 L CNN
+F 1 "R_7.5M" H 3270 3355 50  0000 L CNN
+F 2 "footprints:R_0805_OEM" H 2100 3700 50  0001 L CNN
+F 3 "https://www.yageo.com/upload/media/product/productsearch/datasheet/rchip/PYu-RC_Group_51_RoHS_L_11.pdf" H 2100 3800 50  0001 L CNN
+F 4 "https://www.digikey.com/product-detail/en/yageo/RC0805FR-077M5L/311-7-50MCRTR-ND/728117" H 2100 3900 60  0001 L CNN "PurchasingLink"
+	1    3200 3400
+	1    0    0    -1
+$EndComp
 $EndSCHEMATC

Commit message: fixed
Parts:
- removed C1: C_4.7uF_25V, footprints:C_0805_OEM, symbol AE-001_Analog_Sensing_Supply-rescue:C_4.7uF_25V-Formula
- removed C2: C_10nF, footprints:C_0805_OEM, symbol AE-001_Analog_Sensing_Supply-rescue:C_10nF-Formula
- removed C3: C_10uF, footprints:C_0805_OEM, symbol AE-001_Analog_Sensing_Supply-rescue:C_10uF-Formula
- removed D1: CDBA140-G, symbol AE-001_Analog_Sensing_Supply-rescue:CDBA140-G-Formula
- removed L1: L_2.2uH, symbol AE-001_Analog_Sensing_Supply-rescue:L_2.2uH-Formula
- removed R1: R_7.5M, footprints:R_0805_OEM, symbol AE-001_Analog_Sensing_Supply-rescue:R_7.5M-Formula
- removed R2: R_49.9K, footprints:R_0805_OEM, symbol AE-001_Analog_Sensing_Supply-rescue:R_49.9K-Formula
- removed R3: R_9.53K, footprints:R_0805_OEM, symbol AE-001_Analog_Sensing_Supply-rescue:R_9.53K-Formula
- removed U1: AOZ1280, symbol AE-001_Analog_Sensing_Supply-rescue:AOZ1280-Formula
- added C1: C_4.7uF_25V, footprints:C_0805_OEM, symbol formula:C_4.7uF_25V
- added C2: C_10nF, footprints:C_0805_OEM, symbol formula:C_10nF
- added C3: C_10uF, footprints:C_0805_OEM, symbol formula:C_10uF
- added D1: CDBA140-G, symbol formula:CDBA140-G
- added L1: L_2.2uH, symbol formula:L_2.2uH
- added R1: R_7.5M, footprints:R_0805_OEM, symbol formula:R_7.5M
- added R2: R_49.9K, footprints:R_0805_OEM, symbol formula:R_49.9K
- added R3: R_9.53K, footprints:R_0805_OEM, symbol formula:R_9.53K
- added U1: AOZ1280, symbol formula:AOZ1280

Commit message: PS2 and PS4 layout
Parts:
- D1: footprint (none) -> footprints:DO-214AC
- L1: footprint (none) -> footprints:BRL3225
- U1: footprint (none) -> footprints:SOT-23-6_OEM
Changed lines of the file:
@@
 $Descr A4 11693 8268
 encoding utf-8
-Sheet 3 4
+Sheet 1 1
 Title "Asynchronous Buck"
 Date ""
@@
 	4700 3550 5150 3550
 Connection ~ 4700 3550
-Text Label 6550 3550 0    50   ~ 0
-VOUT
 Wire Wire Line
 	4700 3100 4700 3550
@@
 F 0 "U1" H 3550 3200 50  0000 R CNN
 F 1 "AOZ1280" H 3600 3100 50  0000 R CNN
-F 2 "" H 4150 3850 50  0001 C CNN
+F 2 "footprints:SOT-23-6_OEM" H 4150 3850 50  0001 C CNN
 F 3 "http://aosmd.com/res/data_sheets/AOZ1280CI.pdf" H 4150 3850 50  0001 C CNN
 F 4 "https://www.digikey.com/product-detail/en/alpha-omega-semiconductor-inc/AOZ1280CI/785-1277-1-ND/2769845" H 3350 4150 50  0001 C CNN "Purchasing Link"
@@
 F 0 "D1" V 4654 3879 50  0000 L CNN
 F 1 "CDBA140-G" V 4745 3879 50  0000 L CNN
-F 2 "" H 4600 3800 50  0001 C CNN
+F 2 "footprints:DO-214AC" H 4600 3800 50  0001 C CNN
 F 3 "https://media.digikey.com/pdf/Data%20Sheets/Comchip%20PDFs/CDBA120-G~CDBA1100-G.pdf" H 4700 3900 50  0001 C CNN
 F 4 "https://www.digikey.in/product-detail/en/comchip-technology/CDBA140-G/641-1015-1-ND/1121137" H 5000 4200 60  0001 C CNN "PurchasingLink"
@@
 F 0 "L1" V 5435 3550 50  0000 C CNN
 F 1 "L_2.2uH" V 5344 3550 50  0000 C CNN
-F 2 "" H 5180 3490 50  0001 C CNN
+F 2 "footprints:BRL3225" H 5180 3490 50  0001 C CNN
 F 3 "https://ds.yuden.co.jp/TYCOMPAS/ut/detail?pn=BRL3225T2R2M%20%20&u=M" H 5280 3590 50  0001 C CNN
 F 4 "https://www.digikey.com/product-detail/en/taiyo-yuden/BRL3225T2R2M/587-2165-1-ND/2002863" H 5680 3990 60  0001 C CNN "PurchasingLink"
@@
 F 1 "C_10uF" H 6215 3805 50  0000 L CNN
 F 2 "footprints:C_0805_OEM" H 6138 4400 50  0001 C CNN
-F 3 "http://www.samsungsem.com/kr/support/product-search/mlcc/__icsFiles/afieldfile/2018/06/20/CL21A106KPFNNNE.pdf" H 6125 4650 50  0001 C CNN
+F 3 "https://media.digikey.com/pdf/Data%20Sheets/Samsung%20PDFs/CL_Series_MLCC_ds.pdf" H 6125 4650 50  0001 C CNN
 F 4 "DK" H 6100 3850 60  0001 C CNN "MFN"
 F 5 "1276-1052-1-ND" H 6100 4550 60  0001 C CNN "MPN"
@@
 Wire Wire Line
 	5550 4250 6100 4250
+Text Label 6550 3550 0    50   ~ 0
+VOUT
 $EndSCHEMATC
