File: AE-001_Analog_Sensing_Supply/PS1.sch (KiCad schematic (older format))
At the start: 8 parts, among them U1 lm2841Y

Commit message: updated layout for lm2841Y switching regulator, needs review
Parts:
- removed C1: C_0.1uF_0603, footprints:C_0603_1608Metric, symbol formula:C_0.1uF_0603
- removed C2: C_10uF, footprints:C_0805_OEM, symbol formula:C_10uF
- removed R1: R_10K, footprints:R_0805_OEM, symbol formula:R_10K
- removed R2: R_55.35K, footprints:R_0805_OEM, symbol formula:R_10K
- added C1: C_0.15uF, footprints:C_0805_OEM, symbol formula:C_0.1uF
- added C2: C_47uF, footprints:C_0805_OEM, symbol formula:C_47uF
- added R1: R_1.02K, footprints:R_0805_OEM, symbol formula:R_1K_0.1
- added R2: R_5.62K, footprints:R_0805_OEM, symbol formula:R_1K_0.1
- U1: footprint (none) -> footprints:LM2841Y
Other:
- moved on the sheet: D1
Changed lines of the file:
@@
 EESchema Schematic File Version 4
+LIBS:PS1-cache
 EELAYER 30 0
 EELAYER END
@@
 F 0 "U1" H 5900 3717 50  0000 C CNN
 F 1 "lm2841Y" H 5900 3626 50  0000 C CNN
-F 2 "" H 5900 3600 50  0001 C CNN
+F 2 "footprints:LM2841Y" H 5900 3600 50  0001 C CNN
 F 3 "" H 5900 3600 50  0001 C CNN
 	1    5900 3450
@@
 Wire Wire Line
 	6300 3650 6500 3650
-$Comp
-L formula:R_10K R1
-U 1 1 5F2E1F0A
-P 6500 3800
-F 0 "R1" H 6570 3846 50  0000 L CNN
-F 1 "R_10K" H 6570 3755 50  0000 L CNN
-F 2 "footprints:R_0805_OEM" H 6430 3800 50  0001 C CNN
-F 3 "http://www.bourns.com/data/global/pdfs/CRS.pdf" H 6580 3800 50  0001 C CNN
-F 4 "DK" H 6500 3800 60  0001 C CNN "MFN"
-F 5 "CRS0805-FX-1002ELFCT-ND" H 6500 3800 60  0001 C CNN "MPN"
-F 6 "https://www.digikey.com/products/en?keywords=CRS0805-FX-1002ELFCT-ND" H 6980 4200 60  0001 C CNN "PurchasingLink"
-	1    6500 3800
-	1    0    0    -1
-$EndComp
-$Comp
-L formula:R_10K R2
-U 1 1 5F2E23B1
-P 6650 3650
-F 0 "R2" V 6443 3650 50  0000 C CNN
-F 1 "R_55.35K" V 6534 3650 50  0000 C CNN
-F 2 "footprints:R_0805_OEM" H 6580 3650 50  0001 C CNN
-F 3 "http://www.bourns.com/data/global/pdfs/CRS.pdf" H 6730 3650 50  0001 C CNN
-F 4 "DK" H 6650 3650 60  0001 C CNN "MFN"
-F 5 "CRS0805-FX-1002ELFCT-ND" H 6650 3650 60  0001 C CNN "MPN"
-F 6 "https://www.digikey.com/products/en?keywords=CRS0805-FX-1002ELFCT-ND" H 7130 4050 60  0001 C CNN "PurchasingLink"
-	1    6650 3650
-	0    1    1    0
-$EndComp
-Connection ~ 6500 3650
-Wire Wire Line
-	5900 3950 6500 3950
 Wire Wire Line
 	5900 3850 5900 3950
-Wire Wire Line
-	7500 3950 7500 3450
 Wire Wire Line
 	5500 3650 5350 3650
@@
 Text Label 5150 3450 2    50   ~ 0
 VIN
-$Comp
-L formula:C_0.1uF_0603 C1
-U 1 1 5F4863C6
-P 6450 3100
-F 0 "C1" V 6198 3100 50  0000 C CNN
-F 1 "C_0.1uF_0603" V 6289 3100 50  0000 C CNN
-F 2 "footprints:C_0603_1608Metric" H 6488 2950 50  0001 C CNN
-F 3 "https://media.digikey.com/pdf/Data%20Sheets/Samsung%20PDFs/CL_Series_MLCC_ds.pdf" H 6475 3200 50  0001 C CNN
-F 4 "DK" H 6450 3100 60  0001 C CNN "MFN"
-F 5 "1276-6582-1-ND" H 6450 3100 60  0001 C CNN "MPN"
-F 6 "https://www.digikey.com/product-detail/en/samsung-electro-mechanics/CL10B104KO8WPNC/1276-6582-1-ND/5961441" H 6875 3600 60  0001 C CNN "PurchasingLink"
-	1    6450 3100
-	0    1    1    0
-$EndComp
 Wire Wire Line
 	6300 3100 6300 3450
@@
 Wire Wire Line
 	6600 3550 6600 3100
-Connection ~ 6600 3100
-$Comp
-L formula:C_10uF C2
-U 1 1 5F4881AF
-P 7500 3350
-F 0 "C2" H 7615 3446 50  0000 L CNN
-F 1 "C_10uF" H 7615 3355 50  0000 L CNN
-F 2 "footprints:C_0805_OEM" H 7538 3950 50  0001 C CNN
-F 3 "http://www.samsungsem.com/kr/support/product-search/mlcc/__icsFiles/afieldfile/2018/06/20/CL21A106KPFNNNE.pdf" H 7525 4200 50  0001 C CNN
-F 4 "DK" H 7500 3400 60  0001 C CNN "MFN"
-F 5 "1276-1052-1-ND" H 7500 4100 60  0001 C CNN "MPN"
-F 6 "https://www.digikey.com/product-detail/en/samsung-electro-mechanics/CL21A106KPFNNNE/1276-1052-1-ND/3889138" H 7925 3850 60  0001 C CNN "PurchasingLink"
-	1    7500 3350
-	1    0    0    -1
-$EndComp
-Connection ~ 6500 3950
-Wire Wire Line
-	6800 3650 7300 3650
-Wire Wire Line
-	7300 3650 7300 3100
-Wire Wire Line
-	6500 3950 7500 3950
 $Comp
 L formula:L_15uH L1
@@
 	1    0    0    -1
 $EndComp
-Wire Wire Line
-	7300 3100 7500 3100
-Wire Wire Line
-	7500 3100 7500 3150
-Connection ~ 7300 3100
-Wire Wire Line
-	7500 3100 7600 3100
-Connection ~ 7500 3100
 Text Label 7600 3100 0    50   ~ 0
 5V_out
-Wire Wire Line
-	6600 3100 6850 3100
-Text Label 6850 3400 0    50   ~ 0
-GND
 Wire Wire Line
 	5900 3950 5200 3950
@@
 L Diode:MBR0530 D1
 U 1 1 5F492AFD
-P 6850 3250
-F 0 "D1" V 6804 3329 50  0000 L CNN
-F 1 "MBR0530" V 6895 3329 50  0000 L CNN
-F 2 "Diode_SMD:D_SOD-123" H 6850 3075 50  0001 C CNN
-F 3 "http://www.mccsemi.com/up_pdf/MBR0520~MBR0580(SOD123).pdf" H 6850 3250 50  0001 C CNN
-	1    6850 3250
+P 7100 3250
+F 0 "D1" V 7054 3329 50  0000 L CNN
+F 1 "MBR0530" V 7145 3329 50  0000 L CNN
+F 2 "Diode_SMD:D_SOD-123" H 7100 3075 50  0001 C CNN
+F 3 "http://www.mccsemi.com/up_pdf/MBR0520~MBR0580(SOD123).pdf" H 7100 3250 50  0001 C CNN
+	1    7100 3250
 	0    1    1    0
 $EndComp
-Connection ~ 6850 3100
 Wire Wire Line
-	6850 3100 7100 3100
+	5900 3950 6500 3950
+Text Label 6850 3650 0    50   ~ 0
+5V_out
+Connection ~ 7100 3100
+$Comp
+L formula:R_1K_0.1 R2
+U 1 1 5F51E4B6
+P 6700 3650
+F 0 "R2" V 6907 3650 50  0000 C CNN
+F 1 "R_5.62K" V 6816 3650 50  0000 C CNN
+F 2 "footprints:R_0805_OEM" H 6630 3650 50  0001 C CNN
+F 3 "https://industrial.panasonic.com/cdbs/www-data/pdf/RDM0000/AOA0000C307.pdf" H 6780 3650 50  0001 C CNN
+F 4 "DK" H 6700 3650 60  0001 C CNN "MFN"
+F 5 "P1.0KDACT-ND" H 6700 3650 60  0001 C CNN "MPN"
+F 6 "https://www.digikey.com/product-detail/en/panasonic-electronic-components/ERA-6AEB102V/P1.0KDACT-ND/1465947" H 7180 4050 60  0001 C CNN "PurchasingLink"
+	1    6700 3650
+	0    -1   -1   0
+$EndComp
+$Comp
+L formula:R_1K_0.1 R1
+U 1 1 5F520CA4
+P 6500 3800
+F 0 "R1" H 6430 3754 50  0000 R CNN
+F 1 "R_1.02K" H 6430 3845 50  0000 R CNN
+F 2 "footprints:R_0805_OEM" H 6430 3800 50  0001 C CNN
+F 3 "https://industrial.panasonic.com/cdbs/www-data/pdf/RDM0000/AOA0000C307.pdf" H 6580 3800 50  0001 C CNN
+F 4 "DK" H 6500 3800 60  0001 C CNN "MFN"
+F 5 "P1.0KDACT-ND" H 6500 3800 60  0001 C CNN "MPN"
+F 6 "https://www.digikey.com/product-detail/en/panasonic-electronic-components/ERA-6AEB102V/P1.0KDACT-ND/1465947" H 6980 4200 60  0001 C CNN "PurchasingLink"
+	1    6500 3800
+	-1   0    0    1
+$EndComp
+Wire Wire Line
+	6600 3100 7100 3100
+Wire Wire Line
+	6550 3650 6500 3650
+Connection ~ 6500 3650
+Wire Wire Line
+	7100 3400 7100 3950
+Connection ~ 7100 3950
+Wire Wire Line
+	7300 3100 7550 3100
+$Comp
+L formula:C_0.1uF C1
+U 1 1 5F5253C2
+P 6450 3100
+F 0 "C1" V 6198 3100 50  0000 C CNN
+F 1 "C_0.15uF" V 6289 3100 50  0000 C CNN
+F 2 "footprints:C_0805_OEM" H 6488 2950 50  0001 C CNN
+F 3 "http://datasheets.avx.com/X7RDielectric.pdf" H 6475 3200 50  0001 C CNN
+F 4 "DK" H 6450 3100 60  0001 C CNN "MFN"
+F 5 "478-3352-1-ND" H 6450 3100 60  0001 C CNN "MPN"
+F 6 "https://www.digikey.com/products/en?keywords=478-3352-1-ND" H 6875 3600 60  0001 C CNN "PurchasingLink"
+	1    6450 3100
+	0    1    1    0
+$EndComp
+Connection ~ 6600 3100
+Wire Wire Line
+	7550 3100 7550 3450
+Connection ~ 7550 3100
+Wire Wire Line
+	7550 3100 7600 3100
+$Comp
+L formula:C_47uF C2
+U 1 1 5F525E92
+P 7550 3600
+F 0 "C2" H 7665 3646 50  0000 L CNN
+F 1 "C_47uF" H 7665 3555 50  0000 L CNN
+F 2 "footprints:C_0805_OEM" H 7588 3450 50  0001 C CNN
+F 3 "http://www.samsungsem.com/kr/support/product-search/mlcc/__icsFiles/afieldfile/2018/06/22/CL21A476MQYNNNG.pdf" H 7575 3700 50  0001 C CNN
+F 4 "DK" H 7550 3600 60  0001 C CNN "MFN"
+F 5 "1276-6467-1-ND" H 7550 3600 60  0001 C CNN "MPN"
+F 6 "https://www.digikey.com/product-detail/en/samsung-electro-mechanics/CL21A476MQYNNNG/1276-6467-1-ND/5958095" H 7975 4100 60  0001 C CNN "PurchasingLink"
+	1    7550 3600
+	1    0    0    -1
+$EndComp
+Wire Wire Line
+	7100 3950 7550 3950
+Wire Wire Line
+	7550 3750 7550 3950
+Connection ~ 6500 3950
+Wire Wire Line
+	6500 3950 7100 3950
 $EndSCHEMATC
